File: KiCAD/cafeFlex.kicad_sch (KiCad schematic)
At the start: 7 parts, among them J18 503398-1892, U1 K9K8G08U1D

Commit message: update schem+board
Parts:
- added J1: 2.4GHz Wi-Fi B2B, cafeflex:wificonn, symbol Connector_Generic:Conn_02x10_Counter_Clockwise
- added TP1, TP2, TP3: TestPoint, TestPoint:TestPoint_Pad_1.5x1.5mm, symbol Connector:TestPoint
Connections:
- net +3V3: now also J1.11 (Pin_11), J1.12 (Pin_12), J1.14 (Pin_14), J1.7 (Pin_7), J1.9 (Pin_9), TP1.1, TP3.1; no longer R2.1
- net GND: now also J18.10 (DETECT_SWITCH), J18.11, J18.12, J18.13, J18.14, J18.9 (DETECT_LEVER), J1.1 (GND), J1.13 (Pin_13), J1.15 (Pin_15), J1.17 (Pin_17), J1.20 (Pin_20), J1.4 (Pin_4), J1.6 (Pin_6), J1.8 (Pin_8), TP2.1
- new net D1: J1.19 (Pin_19)
- new net D2: J1.16 (Pin_16)
- new net D3: J1.3 (Pin_3)
- new net D4: J1.18 (Pin_18)
- new net D5: J1.5 (Pin_5)
- new net D6: J1.2 (Pin_2)
- no-connect marks 0 -> 1

Commit message: finalize, add gerbers
Connections:
- net +3V3: now also R2.1
Changed lines of the file:
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@@
+	(symbol
+		(lib_id "power:+3V3")
+		(at 157.48 52.07 0)
+		(unit 1)
+		(exclude_from_sim no)
+		(in_bom yes)
+		(on_board yes)
+		(dnp no)
+		(property "Reference" "#PWR09"
+			(at 157.48 55.88 0)
+			(effects
+				(font
+					(size 1.27 1.27)
+				)
+				(hide yes)
+			)
+		)
+		(property "Value" "+3V3"
+			(at 157.48 48.26 0)
+			(effects
+				(font
+					(size 1.27 1.27)
+				)
+			)
+		)
+		(property "Footprint" ""
+			(at 157.48 52.07 0)
+			(effects
+				(font
+					(size 1.27 1.27)
+				)
+				(hide yes)
+			)
+		)
+		(property "Datasheet" ""
+			(at 157.48 52.07 0)
+			(effects
+				(font
+					(size 1.27 1.27)
+				)
+				(hide yes)
+			)
+		)
+		(property "Description" ""
+			(at 157.48 52.07 0)
+			(effects
+				(font
+					(size 1.27 1.27)
+				)
+				(hide yes)
+			)
+		)
+		(pin "1"
+		)
+		(instances
+			(project "cafeFlex"
+				(path "/b19cb028-dbde-4027-a5b8-5e978264ede3"
+					(reference "#PWR09")
+					(unit 1)
+				)
+			)
+		)
+	)
 	(symbol
 		(lib_id "power:+3V3")
